File: TMS2V.kicad_pcb (KiCad board)
At the start: 2 copper layers, 37 parts, among them J1 TMS9918A Socket, J3 RGB Out, J4 RGB Header, Q1 BC547, Q2 BC547, Q3 BC547, Q4 BC547, U1 V9938, U2 D41464, U3 D41464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

Commit message: Initial PCB layout
Parts:
- moved C3 109.5 mm to (186.0, 80.0), turned to 180 degrees
- moved C2 109.1 mm to (186.0, 76.8), turned to 180 degrees
- moved R8 100.3 mm to (179.7, 149.2)
- moved R7 100.2 mm to (179.7, 144.1)
- moved C6 97.3 mm to (181.0, 109.2)
- moved C4 92.7 mm to (165.1, 83.1), turned to 90 degrees
- moved C8 91.2 mm to (181.1, 137.8)
- moved R6 89.8 mm to (167.0, 149.2)
- moved R5 89.6 mm to (167.0, 144.1)
- moved R2 86.9 mm to (165.1, 85.7), turned to -90 degrees
- moved C5 85.8 mm to (170.2, 109.2)
- moved R4 84.6 mm to (165.1, 123.8), turned to 90 degrees
- moved R1 84.5 mm to (165.1, 95.9), turned to -90 degrees
- moved R3 84.2 mm to (165.1, 113.7), turned to 90 degrees
- moved C7 79.8 mm to (170.3, 137.8)
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Other:
- board outline added: 73 x 80.6 mm
- board text added: "GND"
- board text added: "Gavin Tersteeg"
- board text added: "MODE1"
- board text added: "Rev. 0"
- board text added: "TMS2V"

Commit message: Generated gerbers
Parts:
- moved U1 0.69 mm to (152.4, 103.1)
Routing:
- net GND: track 0.00 -> 315.2 mm
- net +5V: track 0.00 -> 182.5 mm
- net /VA2: track 0.00 -> 106.4 mm, vias 0 -> 1
- net /VA1: track 0.00 -> 103.4 mm, vias 0 -> 1
- net /VA7: track 0.00 -> 103.3 mm
- net /VA0: track 0.00 -> 81.4 mm, vias 0 -> 1
- net Net-(Q1-B): track 0.00 -> 79.9 mm
- net /VA3: track 0.00 -> 72.8 mm
- net Net-(U1-*RAS): track 0.00 -> 70.3 mm
- net Net-(U1-CSYNC): track 0.00 -> 69.7 mm
- net Net-(Q2-B): track 0.00 -> 68.5 mm
- net /VA4: track 0.00 -> 65.7 mm
- net /VA5: track 0.00 -> 65.1 mm
- net Net-(U2-*RAS): track 0.00 -> 64.6 mm
- net /VA6: track 0.00 -> 62.0 mm, vias 0 -> 1
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- added copper zone on B.Cu, net GND
- added copper zone on F.Cu, net GND
